File: kicad/superball_powerboard.sch (KiCad schematic (older format))
At the start: 62 parts

Commit message: almost done with the schematic. still need to add the connectors and the 5.5V gate drivers.
Parts:
- added C? (x11): 100nF, symbol C
- added C?: 10uF 16V, symbol C
- added C?: 100nF, 100nF, symbol C
- added C? (x2): C, symbol C
- added C?: 10uF, symbol C
- added D?: MC06CF 004, 0603, symbol R
- added D?: VBUS05L1-DD1, 0402, symbol R
- added D? (x2): LED, symbol LED
- added JP?: PINHD-1X5, pinhead-1X05, symbol PINHD-1X5
- added JP? (x2): PINHD-1X2, pinhead-1X02, symbol PINHD-1X2
- added JP?: BZW06-26B, pinhead-1X02, symbol PINHD-1X2
- added JP?: PINHD-1X10, pinhead-1X10, symbol PINHD-1X10
- added JP?: ANT, pinhead-1X01, symbol PINHD-1X1
- added L?: FERRITE, 0805, symbol INDUCTOR
- added Q?: MCP73832, SOT_23_5, symbol MCP73831
- added Q?: RF803D, SOIC_8, symbol RF803D
- added R? (x7): 10000, symbol R
- added R?: 470, symbol R
- added R? (x2): 4700, symbol R
- added R?: FUSE 8A, 1206, symbol R
- added R? (x4): 1000, symbol R
- added R?: INF, symbol R
- added R?: 0, 1210, symbol R
- added R?: R, symbol R
- added R?: 100K, symbol R
- added R?: 2200, symbol R
- added R?: 0, symbol R
- added R? (x2): 50K, symbol R
- added U?: LDO 3V3 SOT-223, symbol LD1117
- added U?: SI1970DH, MODULE, symbol SI1970DH
- R?: value R -> INF
Connections:
- net labels added: AF_GND, AF_VCC, AN11, AN6, AN7, AN8, BUZZER, B_LED, G_LED, MCLR, OP1, OP2, OP3, PGEC, PGED, RF_ANT, RF_DOUT, RF_GND, RF_LEARN, RF_SERIAL, RF_VCC, R_LED, SCL, SDA, STATUS_LED, SWITCH_ON, Tensegrity SUPERball power board, VBACKUP_CHARGE_EN, VBACKUP_STAT, VBAT_IN
- wire segments 157 -> 364
Other:
- note added: "1206SFS800F/24"
- note added: "OFF\n"
- note added: "ONE PIN switching"
- note added: "ON\n"
- note added: "POWER LEDS\n"
- note added: "UART\n"
- note added: "default: VBACKUP enabled!!!\n"
- note added: "monitors 5.5V line (should be stable...)\n"
- note added: "monitors backup battery voltage\n"
- note added: "muhahahaa"
- note removed: "TODO: voltage divider backup battery \n"
- note removed: "add voltage divider for main battery 5.5V\n"
- moved on the sheet: C?, JP?, Q?, U?

Commit message: schematic is semi-finished. Needs some cleanup
Parts:
- removed R?: 0, 1210, symbol R
- removed U?: SI1970DH, MODULE, symbol SI1970DH
- added D? (x7): LED, symbol LED
- added J? (x7): MICROCLASP_HDRX2, symbol MICROCLASP_HDRX2
- added R? (x4): 470, symbol R
- added R? (x3): 1K, symbol R
- added R?: 5K, symbol R
- added U?: RGB_LED, MODULE, symbol RGB_LED
- D?: footprint (none) -> 0805
- R?: value 13000 -> 13K
- R? (x2): value 2200 -> 2K2
- R?: value 30000 -> 30K
- R? (x2): value 5000 -> 5K
- R? (x8): value 10000 -> 10K
- R? (x2): value 4700 -> 4K7
- R? (x4): value 1000 -> 1K
- R?: value R -> 470
Connections:
- net labels added: EN_VBACKUP_5V5, EN_VBAT_5V5
- wire segments 364 -> 362
Other:
- note added: "Break out pins\n"
- note removed: "ONE PIN switching"
- note removed: "UART\n"

Commit message: finished schematic
Parts:
- removed J?: MICROCLASP_HDRX2, symbol MICROCLASP_HDRX2
- removed JP?: PINHD-1X2, pinhead-1X02, symbol PINHD-1X2
- removed U?: RGB_LED, MODULE, symbol RGB_LED
- added C19: 100nF, symbol C
- added J1, J2: MICROCLASP_HDRX3, symbol MICROCLASP_HDRX3
- added J8: MICROCLASP_HDRX2, symbol MICROCLASP_HDRX2
- added JP4: PINHD-2X6, pinhead-2X06, symbol PINHD-2X6
- added JP5: PINHD-1X2, pinhead-1X02, symbol PINHD-1X2
- added Q12, Q13: LTC1982, SOT23, symbol LTC1982
- added Q14, Q15: FDS6898AZ, SO_8, symbol FDS6898AZ
- added R35: 1K, symbol R
- added R37, R38, R39, R40: 50K, symbol R
- C36: renamed from C?; value C -> 100nF
- C37: renamed from C?; value C -> 10uF
- C7: renamed from C?; value 0.1uF 50V -> 100nF 50V
- R10: renamed from R?; value 30K -> 50K
- R36: renamed from R?; value R -> 120
- gave numbers to parts that had none: 126
Connections:
- net labels added: EN_OUT_1, EN_OUT_2, EN_OUT_3, EN_OUT_4, EX_1, EX_10, EX_2, EX_3, EX_4, EX_5, EX_6, EX_7, EX_8, EX_9, OUT_1, OUT_2, OUT_3, OUT_4
- wire segments 362 -> 415
Other:
- note removed: "Break out pins\n"
- note removed: "POWER LEDS\n"
- note removed: "TODO: Make this bridgeable (DC/DC module)\n"
- note removed: "allow single pin switching + two pin switching of 5.5\n"
- moved on the sheet: C36, C37, D10, D12, D4, D5, D6, D7, D8, D9, JP1, L3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

Commit message: finished schematic, started pcb layout
Parts:
- removed D3: VS-MBRB1635PBF, symbol VS-MBRB1635PBF
- added D3: PDS1040L, symbol PDS1040L
- JP2, JP3: value PINHD-1X2 -> MICROCLASP_HDRX2; symbol PINHD-1X2 -> MICROCLASP_HDRX2
Connections:
- wire segments 415 -> 416
Other:
- note added: "24V kill switch\n"
- note added: "24V->5.5V DC/DC converter (4A)\n"
- note added: "3V-4.2V -> 5.5V DC/DC converter (4A)"
- note added: "5.5V->3.3V LDO\n"
- note added: "backup battery charger\n"
- note added: "blfnars"
- note added: "breakout"
- note added: "programmer"
- note added: "switch between boost and buck converters"
- note added: "switches to enable/disable 5.5V power outputs\n"
- note added: "various analog sensors: current, voltage,..."

Commit message: connected VMOTOR_EN to pin of uC
Parts:
- added R55, R56: 10K, symbol R
Connections:
- wire segments 416 -> 423

Commit message: did initial placement of the components on the pcb
Parts:
- removed C15: 10uF, symbol C
- removed R10, R37, R38, R39, R40: 50K, symbol R
- removed R11: 5K, symbol R
- removed R22: INF, symbol R
- removed R42: 0, symbol R
- R1: value 5K -> 10K
- R5: value INF -> 50K
Connections:
- net labels added: EN_MOTOR_CURRENT, MOTOR_CURRENT_FLT
- wire segments 423 -> 413
Other:
- moved on the sheet: R17

Commit message: fixed a few bugs in the schematic and started preliminary routing
Parts:
- removed D5: LED, symbol LED
- removed R21: 10K, symbol R
- removed R24: 5K, symbol R
- removed U2: CSD16323Q3, symbol CSD16323Q3
- removed U5: LDO 3V3 SOT-223, symbol LD1117
- added C15: 100nF, symbol C
- added Q17: PSMN013-80YS, SOT669, symbol PSMN013-80YS
- added R10: 10K, symbol R
- added R11: 1K, symbol R
- added U5: MCP1700, symbol MCP1700
Connections:
- net labels added: VMOTOR_V
- wire segments 413 -> 485
Other:
- moved on the sheet: C37

Commit message: finished routing (preliminary). Added a current sensor for the 5.5V line.
Parts:
- removed C36: 100nF, symbol C
- added C38: 100nF, symbol C
- added D5: ZENER, 403A−03, symbol ZENER
- added JP13: PINHD-1X8, pinhead-1X08, symbol PINHD-1X8
- added JP14: PINHD-1X2, pinhead-1X02, symbol PINHD-1X2
- added R21: 0.02, SN1206, symbol R
- added U2: INA197, symbol INA197
- R18, R3: value 10K -> 50K
Connections:
- net labels added: 5V5_FUSE, 5V5_MERGE, 5V_CUR, VBACKUP_SW, VBAT_HF_SW, VBAT_SW
- wire segments 485 -> 466
