File: kicad/superball_powerboard.sch (KiCad schematic (older format))
At the start: 147 parts, among them J1 MICROCLASP_HDRX3, J2 MICROCLASP_HDRX3, J3 MICROCLASP_HDRX2, J4 MICROCLASP_HDRX2, J5 MICROCLASP_HDRX2, J6 MICROCLASP_HDRX2, J7 MICROCLASP_HDRX2, J8 MICROCLASP_HDRX2, J9 MICROCLASP_HDRX2, Q1 MCP73832, Q10 FDS6898AZ, Q11 FDS6898AZ, Q12 LTC1982, Q13 LTC1982, Q14 FDS6898AZ, Q15 FDS6898AZ, Q16 RF803D, Q17 PSMN013-80YS, Q2 LM3478, Q3 TPS54540, Q4 LT1910, Q5 0S102011MA1QN1, Q6 PSMN013-80YS, Q7 PSMN013-80YS, Q8 LTC1982, Q9 ACS711KLCTR-12AB-T, U1 SI1970DH, U2 INA197, U3 SN65HVD232, U4 DSPIC33E128MC506, U5 MCP1700

Commit message: cleaned up traces, added test pins etc
Parts:
- added R22: 0, symbol R
- added R24: INF, symbol R
- added SW1: SW_PUSH_4, symbol SW_PUSH_4
Connections:
- wire segments 466 -> 477

Commit message: Commit of the gerber files used in fabrication.
Parts:
- renumbered JP12 to LEARN, JP10 to RF
Connections:
- wire segments 477 -> 480
Other:
- moved on the sheet: R35
