File: kicad/superball_powerboard.kicad_pcb (KiCad board)
At the start: 4 copper layers, 100 x 50 mm, 161 parts, among them J1 MICROCLASP_HDRX3, J2 MICROCLASP_HDRX3, J3 MICROCLASP_HDRX2, J4 MICROCLASP_HDRX2, J5 MICROCLASP_HDRX2, J6 MICROCLASP_HDRX2, J7 MICROCLASP_HDRX2, J8 MICROCLASP_HDRX2, J9 MICROCLASP_HDRX2, Q1 MCP73832, Q10 FDS6898AZ, Q11 FDS6898AZ, Q12 LTC1982, Q13 LTC1982, Q14 FDS6898AZ, Q15 FDS6898AZ, Q16 RF803D, Q17 PSMN013-80YS, Q2 LM3478, Q3 TPS54540, Q4 LT1910, Q5 0S102011MA1QN1, Q6 PSMN013-80YS, Q7 PSMN013-80YS, Q8 LTC1982, Q9 ACS711KLCTR-12AB-T, SW1 SW_PUSH_4, U1 SI1970DH, U2 INA197, U3 SN65HVD232, U4 DSPIC33E128MC506, U5 MCP1700

Commit message: cleaned up a few traces
Parts:
- moved U3 0.30 mm to (25.8, 31.5)
- moved C21 0.11 mm to (109.9, 40.8)
Routing:
- net /VMOTOR: track 70.1 -> 20.2 mm
- net /EN_MOTOR_CURRENT: track 68.6 -> 81.1 mm
- net /VBAT_SWITCHED: track 15.2 -> 21.9 mm, vias 0 -> 5
- net /RF_DOUT: track 7.53 -> 13.8 mm
- net /5V5: track 171.2 -> 173.6 mm
- net /SCL: track 27.1 -> 25.0 mm
- net 3V3: track 181.2 -> 183.3 mm
- net /VBAT: track 154.4 -> 156.2 mm, vias 12 -> 17
- net /CAN_H: track 34.5 -> 36.0 mm
- net /CAN_L: track 32.6 -> 33.6 mm
- net /VMOTOR_EN: track 140.6 -> 139.6 mm
- net GND: track 432.5 -> 431.8 mm
- net /EX_6: track 27.3 -> 26.6 mm, vias 1 -> 0
- net /MOTOR_CURRENT_FLT: track 92.6 -> 92.0 mm
- net (no net): vias 0 -> 4
- added copper zone on Inner2.Cu, net /VBAT_SWITCHED
- added copper zone on Inner2.Cu, net /VMOTOR
