File: kicad/superball_powerboard_pmos.sch (KiCad schematic (older format))
At the start: 155 parts, among them J1 MICROCLASP_HDRX3, J2 MICROCLASP_HDRX3, J3 MICROCLASP_HDRX2, J4 MICROCLASP_HDRX2, J5 MICROCLASP_HDRX2, J6 MICROCLASP_HDRX2, J7 MICROCLASP_HDRX2, J8 MICROCLASP_HDRX2, J9 MICROCLASP_HDRX2, Q1 MCP73832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

Commit message: Commit of the gerber files used in fabrication.
Parts:
- gave numbers to parts that had none: 3
Connections:
- wire segments 605 -> 518
Other:
- moved on the sheet: R35
